File: ereader.kicad_pcb (KiCad board)
At the start: 4 copper layers, 66 x 115 mm, 56 parts, among them J1 USB-C-16P, J2 EPD_FPC_24P, J3 FL_FPC_6P, J4 microSD, J5 Battery_1S, SW1 BTN_A, SW2 BTN_B, SW3 BTN_C, SW4 SLLB510200 (PLACEHOLDER-VERIF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, SW5 BOOT, SW6 RESET, U1 ESP32-S3-WROOM-1-N16R8, U2 BQ25628E (PLACEHOLDER-VERIFY), U3 MAX17048 (PLACEHOLDER-VERIFY), U4 LM3630A (PLACEHOLDER-VERIFY), U5 TPS62840 (PLACEHOLDER-VERIFY), U6 USBLC6-2SC6

Commit message: Switches: side-actuated tactiles + real SLLB5 lever land; add schematic
The 3D view showed no lever and top-press buttons because SW1-3/5/6 used the
top-actuated Button_Switch_SMD:SW_SPST_TL3342 stand-in and SW4 was a
PinHeader_1x04 placeholder. With the screen over the whole front and magnets on
the back, only side-actuated, edge-facing controls are reachable.

- Add project footprint library ereader.pretty (registered via new fp-lib-table):
  - Tact_Side_TS1187A_4P_3.5x4.7mm: side-actuated (right-angle) 4-pin SMD tactile
    (TS-1187A / YD-3414 class), actuator on +X face.
  - ALPS_SLLB5_Lever: SLLB5 lever land with pads named CW/CCW/PUSH/COM + 2 lugs.
  Both carry simplified 3D bodies in ereader.3dshapes/*.wrl (scale 0.3937) so they
  render in the 3D viewer without KiCad's stock libraries.
- ereader.kicad_pcb: swap SW1-3/5/6 to the side tactile (rotation 0 so actuators
  face the right edge) and SW4 to the lever (near the left edge); nets preserved.
  SW4's CW/CCW/PUSH/COM now connect to LEV_CW/CCW/PUSH + GND (was unconnected).
- ereader-kicad.net + ereader.cmp: point SW1-6 at the new footprints.
- Add ereader-schematic.md: reviewable subsystem schematic (Mermaid, from the
  connection list) and an explanation of the netlist-first flow / how to draw a
  native Eeschema .kicad_sch (KiCad cannot auto-generate one).
- Docs: update ereader-footprints.md, ereader-README.md, ereader-pcb-design.md,
  README.md, ADR 0008, CHANGELOG. Note SLLB510100 as a pin-compatible alternative.
  Lands are approximate stand-ins - DRC vs the ordered MPN before fab.

Co-Authored-By: Claude Opus 4.8 <noreply@anthropic.com>
Claude-Session: https://claude.ai/code/session_01HmW8HMEGetZ44FEMTwfJYH
Parts:
- SW1, SW2, SW3, SW5, SW6: footprint SW_SPST_TL3342 -> ereader:Tact_Side_TS1187A_4P_3.5x4.7mm
- SW4: value SLLB510200 (PLACEHOLDER-VERIFY) -> SLLB510200; footprint PinHeader_1x04_P2.54mm_Vertical -> ereader:ALPS_SLLB5_Lever
- moved SW4 2.00 mm to (8.00, 46.0), turned to 0 degrees
- turned SW1 to 0 degrees
- turned SW2 to 0 degrees
- turned SW3 to 0 degrees

Commit message: Lock switch footprints to datasheets: WS-TASU tactile + ALPS SLLB5 lever
Rebuilt both project footprints from the manufacturer datasheets supplied by
the user, replacing the approximate stand-ins.

- Tactiles SW1-3/5/6: new ereader:WE_WS-TASU_436351045816 (Wurth WS-TASU
  436351045816, 4.7x3.5mm side push with boss). Land per WE datasheet rev
  001.003: 4 pads 1.2x0.7mm at x=+/-2.8, y=+/-1.35, plus two Ø0.75 boss holes
  on the centreline at y=+/-1.375; pins 1=3 (top) / 2=4 (bottom). Placed at
  rotation 270 so the actuator faces the right board edge. Nets preserved.
- SW4 lever: rebuilt ereader:ALPS_SLLB5_Lever from the ALPS SLLB5 datasheet
  (p.491): 4 signal pads 1.0x1.3mm on 2mm pitch in terminal order
  CW / COM / PUSH / CCW, two Ø1.1 locator holes at x=+/-1.9, and side solder
  lugs; body 9.5x8.8mm. Placed at rotation 90 so the lever faces the left edge.
  Nets unchanged (LEV_CW/CCW/PUSH + COM->GND).
- Replaced the 3D bodies, updated ereader-kicad.net / ereader.cmp footprint ids,
  and refreshed ereader-footprints.md, ereader-pcb-design.md, ADR 0008, CHANGELOG.
  Verified: all six switches on-board, no footprint-origin collisions, PCB
  s-expression balanced.

Lands are datasheet-drawn but should still be DRC'd against the ordered part
before fabrication.

Co-Authored-By: Claude Opus 4.8 <noreply@anthropic.com>
Claude-Session: https://claude.ai/code/session_01HmW8HMEGetZ44FEMTwfJYH
Parts:
- SW1, SW2, SW3, SW5, SW6: footprint ereader:Tact_Side_TS1187A_4P_3.5x4.7mm -> ereader:WE_WS-TASU_436351045816
- turned SW1 to 270 degrees
- turned SW2 to 270 degrees
- turned SW3 to 270 degrees
- turned SW4 to 90 degrees
- turned SW5 to 270 degrees
- turned SW6 to 270 degrees

Commit message: Replace BOOT/RESET tactiles (SW5/SW6) with bare jumper pads (JP5/JP6)
BOOT and RESET are a rarely-used recovery path, so swap the Würth
WS-TASU tactiles for two exposed 2-pad jumpers (ereader:JumperPad_2P_P2.0mm)
at the same board location: momentarily short them with a screwdriver tip
or tweezers to pull IO0/EN low instead of pressing a switch. Drops two
tactile switches from the BOM; same nets, same footprint spot.

Updated the whole netlist-first chain: connection list, schematic,
pcb-design spec, footprints picklist, kicad netlist/.cmp/.kicad_pcb,
placement SVG, ADRs 0004/0008, runbook, and both READMEs.

Co-Authored-By: Claude Sonnet 5 <noreply@anthropic.com>
Claude-Session: https://claude.ai/code/session_01B4v94GAArsLY4TGCiyCJzq
Parts:
- removed SW5: BOOT, ereader:WE_WS-TASU_436351045816
- removed SW6: RESET, ereader:WE_WS-TASU_436351045816
- added JP5: BOOT, ereader:JumperPad_2P_P2.0mm, F.Cu at (58.0, 98.0)
- added JP6: RESET, ereader:JumperPad_2P_P2.0mm, F.Cu at (58.0, 108.0)
Changed lines of the file:
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@@
     )
   )
-  (footprint "ereader:WE_WS-TASU_436351045816" (layer "F.Cu")
+  (footprint "ereader:JumperPad_2P_P2.0mm" (layer "F.Cu")
     (at 58 108 270)
-    (descr "Wurth WS-TASU 436351045816 side-push tact, 4.7x3.5mm, actuator +Y (-> faces board edge at this rotation). Land per WE datasheet; 2x Ø0.75 boss holes. Verify vs datasheet before fab.")
-    (tags "tactile switch side push SMD Wurth WS-TASU boss")
-    (attr smd)
-    (fp_text reference "SW6" (at 0 -2.6 270) (layer "F.SilkS")
-        (effects (font (size 1 1) (thickness 0.15)))
-    )
-    (fp_text value "RESET" (at 0 3.4 270) (layer "F.Fab")
+    (descr "Bare 2-pad exposed jumper (no switch part) - momentarily short with a screwdriver tip or tweezers to pull EN low for RESET. Open circuit in normal use.")
+    (tags "jumper test pad reset bare pads screwdriver")
+    (attr smd)
+    (fp_text reference "JP6" (at 0 -2.6 270) (layer "F.SilkS")
+        (effects (font (size 1 1) (thickness 0.15)))
+    )
+    (fp_text value "RESET" (at 0 2.6 270) (layer "F.Fab")
         (effects (font (size 1 1) (thickness 0.15)))
     )
@@
         (effects (font (size 0.7 0.7) (thickness 0.1)))
     )
-    (fp_line (start -2.35 -1.75) (end 2.35 -1.75) (stroke (width 0.1) (type solid)) (layer "F.Fab"))
-    (fp_line (start 2.35 -1.75) (end 2.35 1.75) (stroke (width 0.1) (type solid)) (layer "F.Fab"))
-    (fp_line (start 2.35 1.75) (end -2.35 1.75) (stroke (width 0.1) (type solid)) (layer "F.Fab"))
-    (fp_line (start -2.35 1.75) (end -2.35 -1.75) (stroke (width 0.1) (type solid)) (layer "F.Fab"))
-    (fp_line (start -0.9 1.75) (end -0.9 2.4) (stroke (width 0.1) (type solid)) (layer "F.Fab"))
-    (fp_line (start -0.9 2.4) (end 0.9 2.4) (stroke (width 0.1) (type solid)) (layer "F.Fab"))
-    (fp_line (start 0.9 2.4) (end 0.9 1.75) (stroke (width 0.1) (type solid)) (layer "F.Fab"))
-    (fp_line (start 0 1.95) (end 0 1.4) (stroke (width 0.12) (type solid)) (layer "F.SilkS"))
-    (fp_line (start -0.15 1.55) (end 0 1.4) (stroke (width 0.12) (type solid)) (layer "F.SilkS"))
-    (fp_line (start 0.15 1.55) (end 0 1.4) (stroke (width 0.12) (type solid)) (layer "F.SilkS"))
-    (fp_line (start -1.9 -1.75) (end -1.9 1.75) (stroke (width 0.12) (type solid)) (layer "F.SilkS"))
-    (fp_line (start 1.9 -1.75) (end 1.9 1.75) (stroke (width 0.12) (type solid)) (layer "F.SilkS"))
-    (fp_circle (center 3.4 2.05) (end 3.5 2.05) (stroke (width 0.2) (type solid)) (fill solid) (layer "F.SilkS"))
-    (fp_line (start -3.6 -2.05) (end 3.6 -2.05) (stroke (width 0.05) (type solid)) (layer "F.CrtYd"))
-    (fp_line (start 3.6 -2.05) (end 3.6 2.7) (stroke (width 0.05) (type solid)) (layer "F.CrtYd"))
-    (fp_line (start 3.6 2.7) (end -3.6 2.7) (stroke (width 0.05) (type solid)) (layer "F.CrtYd"))
-    (fp_line (start -3.6 2.7) (end -3.6 -2.05) (stroke (width 0.05) (type solid)) (layer "F.CrtYd"))
-    (pad "1" smd roundrect (at -2.8 1.35 270) (size 1.2 0.7) (layers "F.Cu" "F.Paste" "F.Mask") (roundrect_rratio 0.25)
+    (fp_line (start -1 -1.9) (end 1 -1.9) (stroke (width 0.1) (type solid)) (layer "F.Fab"))
+    (fp_line (start 1 -1.9) (end 1 1.9) (stroke (width 0.1) (type solid)) (layer "F.Fab"))
+    (fp_line (start 1 1.9) (end -1 1.9) (stroke (width 0.1) (type solid)) (layer "F.Fab"))
+    (fp_line (start -1 1.9) (end -1 -1.9) (stroke (width 0.1) (type solid)) (layer "F.Fab"))
+    (fp_line (start -1.3 -2.2) (end 1.3 -2.2) (stroke (width 0.05) (type solid)) (layer "F.CrtYd"))
+    (fp_line (start 1.3 -2.2) (end 1.3 2.2) (stroke (width 0.05) (type solid)) (layer "F.CrtYd"))
+    (fp_line (start 1.3 2.2) (end -1.3 2.2) (stroke (width 0.05) (type solid)) (layer "F.CrtYd"))
+    (fp_line (start -1.3 2.2) (end -1.3 -2.2) (stroke (width 0.05) (type solid)) (layer "F.CrtYd"))
+    (pad "1" smd rect (at 0 1) (size 1.2 1.2) (layers "F.Cu" "F.Paste" "F.Mask")
       (net 31 "EN"))
-    (pad "1" smd roundrect (at 2.8 1.35 270) (size 1.2 0.7) (layers "F.Cu" "F.Paste" "F.Mask") (roundrect_rratio 0.25)
-      (net 31 "EN"))
-    (pad "2" smd roundrect (at -2.8 -1.35 270) (size 1.2 0.7) (layers "F.Cu" "F.Paste" "F.Mask") (roundrect_rratio 0.25)
+    (pad "2" smd rect (at 0 -1) (size 1.2 1.2) (layers "F.Cu" "F.Paste" "F.Mask")
       (net 5 "GND"))
-    (pad "2" smd roundrect (at 2.8 -1.35 270) (size 1.2 0.7) (layers "F.Cu" "F.Paste" "F.Mask") (roundrect_rratio 0.25)
-      (net 5 "GND"))
-    (pad "" np_thru_hole circle (at 0 1.375) (size 0.75 0.75) (drill 0.75) (layers "*.Cu" "*.Mask"))
-    (pad "" np_thru_hole circle (at 0 -1.375) (size 0.75 0.75) (drill 0.75) (layers "*.Cu" "*.Mask"))
-    (model "${KIPRJMOD}/ereader.3dshapes/WE_WS-TASU_436351045816.wrl"
-    (offset (xyz 0 0 0))
-    (scale (xyz 0.3937 0.3937 0.3937))
-    (rotate (xyz 0 0 0)))
   )
   (footprint "D_SOD-123" (layer "F.Cu")
@@
     )
   )
-  (footprint "ereader:WE_WS-TASU_436351045816" (layer "F.Cu")
+  (footprint "ereader:JumperPad_2P_P2.0mm" (layer "F.Cu")
     (at 58 98 270)
-    (descr "Wurth WS-TASU 436351045816 side-push tact, 4.7x3.5mm, actuator +Y (-> faces board edge at this rotation). Land per WE datasheet; 2x Ø0.75 boss holes. Verify vs datasheet before fab.")
-    (tags "tactile switch side push SMD Wurth WS-TASU boss")
-    (attr smd)
-    (fp_text reference "SW5" (at 0 -2.6 270) (layer "F.SilkS")
-        (effects (font (size 1 1) (thickness 0.15)))
-    )
-    (fp_text value "BOOT" (at 0 3.4 270) (layer "F.Fab")
+    (descr "Bare 2-pad exposed jumper (no switch part) - momentarily short with a screwdriver tip or tweezers to pull IO0 low for BOOT. Open circuit in normal use.")
+    (tags "jumper test pad boot bare pads screwdriver")
+    (attr smd)
+    (fp_text reference "JP5" (at 0 -2.6 270) (layer "F.SilkS")
+        (effects (font (size 1 1) (thickness 0.15)))
+    )
+    (fp_text value "BOOT" (at 0 2.6 270) (layer "F.Fab")
         (effects (font (size 1 1) (thickness 0.15)))
     )
@@
         (effects (font (size 0.7 0.7) (thickness 0.1)))
     )
-    (fp_line (start -2.35 -1.75) (end 2.35 -1.75) (stroke (width 0.1) (type solid)) (layer "F.Fab"))
-    (fp_line (start 2.35 -1.75) (end 2.35 1.75) (stroke (width 0.1) (type solid)) (layer "F.Fab"))
-    (fp_line (start 2.35 1.75) (end -2.35 1.75) (stroke (width 0.1) (type solid)) (layer "F.Fab"))
-    (fp_line (start -2.35 1.75) (end -2.35 -1.75) (stroke (width 0.1) (type solid)) (layer "F.Fab"))
-    (fp_line (start -0.9 1.75) (end -0.9 2.4) (stroke (width 0.1) (type solid)) (layer "F.Fab"))
-    (fp_line (start -0.9 2.4) (end 0.9 2.4) (stroke (width 0.1) (type solid)) (layer "F.Fab"))
-    (fp_line (start 0.9 2.4) (end 0.9 1.75) (stroke (width 0.1) (type solid)) (layer "F.Fab"))
-    (fp_line (start 0 1.95) (end 0 1.4) (stroke (width 0.12) (type solid)) (layer "F.SilkS"))
-    (fp_line (start -0.15 1.55) (end 0 1.4) (stroke (width 0.12) (type solid)) (layer "F.SilkS"))
-    (fp_line (start 0.15 1.55) (end 0 1.4) (stroke (width 0.12) (type solid)) (layer "F.SilkS"))
-    (fp_line (start -1.9 -1.75) (end -1.9 1.75) (stroke (width 0.12) (type solid)) (layer "F.SilkS"))
-    (fp_line (start 1.9 -1.75) (end 1.9 1.75) (stroke (width 0.12) (type solid)) (layer "F.SilkS"))
-    (fp_circle (center 3.4 2.05) (end 3.5 2.05) (stroke (width 0.2) (type solid)) (fill solid) (layer "F.SilkS"))
-    (fp_line (start -3.6 -2.05) (end 3.6 -2.05) (stroke (width 0.05) (type solid)) (layer "F.CrtYd"))
-    (fp_line (start 3.6 -2.05) (end 3.6 2.7) (stroke (width 0.05) (type solid)) (layer "F.CrtYd"))
-    (fp_line (start 3.6 2.7) (end -3.6 2.7) (stroke (width 0.05) (type solid)) (layer "F.CrtYd"))
-    (fp_line (start -3.6 2.7) (end -3.6 -2.05) (stroke (width 0.05) (type solid)) (layer "F.CrtYd"))
-    (pad "1" smd roundrect (at -2.8 1.35 270) (size 1.2 0.7) (layers "F.Cu" "F.Paste" "F.Mask") (roundrect_rratio 0.25)
+    (fp_line (start -1 -1.9) (end 1 -1.9) (stroke (width 0.1) (type solid)) (layer "F.Fab"))
+    (fp_line (start 1 -1.9) (end 1 1.9) (stroke (width 0.1) (type solid)) (layer "F.Fab"))
+    (fp_line (start 1 1.9) (end -1 1.9) (stroke (width 0.1) (type solid)) (layer "F.Fab"))
+    (fp_line (start -1 1.9) (end -1 -1.9) (stroke (width 0.1) (type solid)) (layer "F.Fab"))
+    (fp_line (start -1.3 -2.2) (end 1.3 -2.2) (stroke (width 0.05) (type solid)) (layer "F.CrtYd"))
+    (fp_line (start 1.3 -2.2) (end 1.3 2.2) (stroke (width 0.05) (type solid)) (layer "F.CrtYd"))
+    (fp_line (start 1.3 2.2) (end -1.3 2.2) (stroke (width 0.05) (type solid)) (layer "F.CrtYd"))
+    (fp_line (start -1.3 2.2) (end -1.3 -2.2) (stroke (width 0.05) (type solid)) (layer "F.CrtYd"))
+    (pad "1" smd rect (at 0 1) (size 1.2 1.2) (layers "F.Cu" "F.Paste" "F.Mask")
       (net 30 "IO0_BOOT"))
-    (pad "1" smd roundrect (at 2.8 1.35 270) (size 1.2 0.7) (layers "F.Cu" "F.Paste" "F.Mask") (roundrect_rratio 0.25)
-      (net 30 "IO0_BOOT"))
-    (pad "2" smd roundrect (at -2.8 -1.35 270) (size 1.2 0.7) (layers "F.Cu" "F.Paste" "F.Mask") (roundrect_rratio 0.25)
+    (pad "2" smd rect (at 0 -1) (size 1.2 1.2) (layers "F.Cu" "F.Paste" "F.Mask")
       (net 5 "GND"))
-    (pad "2" smd roundrect (at 2.8 -1.35 270) (size 1.2 0.7) (layers "F.Cu" "F.Paste" "F.Mask") (roundrect_rratio 0.25)
-      (net 5 "GND"))
-    (pad "" np_thru_hole circle (at 0 1.375) (size 0.75 0.75) (drill 0.75) (layers "*.Cu" "*.Mask"))
-    (pad "" np_thru_hole circle (at 0 -1.375) (size 0.75 0.75) (drill 0.75) (layers "*.Cu" "*.Mask"))
-    (model "${KIPRJMOD}/ereader.3dshapes/WE_WS-TASU_436351045816.wrl"
-    (offset (xyz 0 0 0))
-    (scale (xyz 0.3937 0.3937 0.3937))
-    (rotate (xyz 0 0 0)))
   )
   (footprint "ESP32-S3-WROOM-1" (layer "F.Cu")
